Commit message: Add a first fully working Sphero simulation model

File: sphero_description/robots/sphero.gazebo.xacro (robot description, xacro)
@@ -9,10 +9,11 @@
     <maxVel>10.0</maxVel>
     <minDepth>0.0005</minDepth>
+    <gravity>true</gravity>
   </gazebo>
   <gazebo reference="base_rotation_link">
     <kp>100000000.0</kp>
     <kd>10.0</kd>
-    <mu1>10</mu1>
-    <mu2>10</mu2>
+    <mu1>0.4</mu1>
+    <mu2>0.4</mu2>
     <fdir1>1 0 0</fdir1>
     <maxVel>1.0</maxVel>
@@ -22,6 +23,6 @@
     <kp>100000000.0</kp>
     <kd>10.0</kd>
-    <mu1>10</mu1>
-    <mu2>10</mu2>
+    <mu1>0.4</mu1>
+    <mu2>0.4</mu2>
     <fdir1>1 0 0</fdir1>
     <maxVel>1.0</maxVel>
@@ -42,17 +43,18 @@
       <rightJoint>rotation_joint</rightJoint>
       <wheelSeparation>0.0381</wheelSeparation>
-      <wheelDiameter>0.01</wheelDiameter>
-      <torque>20</torque>
-      <commandTopic>/cmd_vel</commandTopic>
-      <odometryTopic>/odom</odometryTopic>
+      <wheelDiameter>0.05</wheelDiameter>
+      <wheelAcceleration>0</wheelAcceleration>
+      <wheelTorque>0.02</wheelTorque>
+      <torque>0.025</torque>
+      <commandTopic>cmd_vel</commandTopic>
+      <odometryTopic>odom</odometryTopic>
       <odometryFrame>/odom_frame</odometryFrame>
+      <positionTopic>pos</positionTopic>
       <publishWheelJointState>true</publishWheelJointState>
-      <odometrySource>world</odometrySource>
+      <publishWheelTF>false</publishWheelTF>
+      <publishTf>1</publishTf> <!-- $$$$$$$$$$$$$$$$$$$$ -->
+      <odometrySource>world</odometrySource>  <!-- $$$$$$$$$$$$$$$$$$$$$ -->
       <robotBaseFrame>base_link</robotBaseFrame>
       <rosDebugLevel>na</rosDebugLevel>
-      <publishWheelTF>true</publishWheelTF>
-      <wheelAcceleration>0</wheelAcceleration>
-      <wheelTorque>5</wheelTorque>
-      <publishTf>1</publishTf>
     </plugin>
   </gazebo>
@@ -60,5 +62,5 @@
   <gazebo>
     <plugin name="gazebo_ros_imu_controller" filename="libgazebo_ros_imu.so">
-      <robotNamespace>/sphero/</robotNamespace>
+      <robotNamespace>/sphero_$(arg prefix)</robotNamespace>
       <topicName>imu/data3</topicName>
       <serviceName>imu/service</serviceName>
@@ -66,13 +68,9 @@
       <!-- <frameId>base_link</frameId> -->
       <gaussianNoise>0</gaussianNoise>
+      <xyzOffset>0 0 0</xyzOffset>
       <rpyOffsets>0 0 0</rpyOffsets>
       <updateRate>50.0</updateRate>
       <alwaysOn>true</alwaysOn>
-      <gaussianNoise>0</gaussianNoise>
-      <xyzOffset>0 0 0</xyzOffset>
-      <rpyOffset>0 0 0</rpyOffset>
-      <!--
-      <frameName>bodyName</frameName>
-  	  -->
+      <!-- <frameName>bodyName</frameName> -->
     </plugin>
   </gazebo>

File: sphero_description/robots/sphero.urdf (robot description, URDF)
Before this commit: robot sphero, 3 links, 2 joints
Links:
- link base_direction_link: mass 0.05 -> 0.01
- link base_link: mass 0.5 -> 0.15; geometry collision sphere radius=0.03; visual sphere radius=0.01
- link base_rotation_link: mass 0.05 -> 0.01; geometry collision sphere radius=0.01; visual sphere radius=0.03
Joints:
- joint direction_joint: axis 1 0 0 -> 0 1 0
- joint rotation_joint: limit lower=-1e+16 upper=1e+16 effort=18.85 velocity=0.2 -> lower=-1e+16 upper=1e+16 effort=18.85 velocity=1.57
